File: board/_autosave-stockton-stem-badge.kicad_pcb (KiCad board)
At the start: 2 copper layers, 50.8 x 50.8 mm, 13 parts, among them J1 ICSP, U1 PIC12LF1501

Commit message: Tweak the silkscreen
- Move various component values into the silkscreen layer
- Label the LEDs by color
Changed lines of the file:
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@@
       (effects (font (size 1 1) (thickness 0.15)))
     )
-    (fp_text value R (at 3.81 0 90) (layer F.Fab)
+    (fp_text value R (at 3.81 0 90) (layer F.SilkS)
       (effects (font (size 1 1) (thickness 0.15)))
     )
@@
       (effects (font (size 1 1) (thickness 0.15)))
     )
-    (fp_text value R (at 3.81 0 90) (layer F.Fab)
+    (fp_text value R (at 3.81 0 90) (layer F.SilkS)
       (effects (font (size 1 1) (thickness 0.15)))
     )
@@
       (effects (font (size 1 1) (thickness 0.15)))
     )
-    (fp_text value R (at 3.81 0 90) (layer F.Fab)
+    (fp_text value R (at 3.81 0 90) (layer F.SilkS)
       (effects (font (size 1 1) (thickness 0.15)))
     )
@@
       (effects (font (size 1 1) (thickness 0.15)))
     )
-    (fp_text value R (at 3.81 0 90) (layer F.Fab)
+    (fp_text value R (at 3.81 0 90) (layer F.SilkS)
       (effects (font (size 1 1) (thickness 0.15)))
     )
